Commit message: fix:将实际抓取的virtual的link位置往手掌中心考

File: src/biped_s4/urdf/biped_s4.urdf (robot description, URDF)
Before this commit: robot biped_s4, 61 links, 60 joints
Joints:
- joint l_hand_end_virtual: origin xyz=0 0 -0.0945 rpy=0 0 0 -> xyz=0 0 -0.1545 rpy=0 0 0
- joint r_hand_end_virtual: origin xyz=0 0 -0.0945 rpy=0 0 0 -> xyz=0 0 -0.1545 rpy=0 0 0
